Commit message: Local planner ve people tracking yapısı eklendi. Topicler ve gerekli parametreler ayarlandı. Arka lidar aktif edildi.

File: wheel_chair/urdf/wheel_chair.urdf (robot description, URDF)
Before this commit: robot wheel_chair, 21 links, 20 joints
Links:
- added link base_footprint
Joints:
- added joint base_joint: type fixed, parent base_footprint, child base_link, origin xyz=0.0 0.0 0.15345 rpy=0 0 0

Commit message: Hatalar düzeltildi.

File: wheel_chair/urdf/wheel_chair.urdf (robot description, URDF)
Before this commit: robot wheel_chair, 22 links, 21 joints
Links:
- added link imu_link
Joints:
- added joint imu_joint: type fixed, parent base_link, child imu_link, origin xyz=-0.032 0 0.068 rpy=0 0 0

Commit message: Proje başarıyla sonuçlanmıştır.

File: wheel_chair/urdf/wheel_chair.urdf (robot description, URDF)
Before this commit: robot wheel_chair, 23 links, 22 joints
Joints:
- joint rp_laser_front_joint: origin xyz=0.72155 0.0046595 -0.074152 rpy=0 0 -0.0013615 -> xyz=0.72155 0.0046595 -0.074152 rpy=0 0 0.01

Commit message: Base footprint ileri kaydırıldı.

File: wheel_chair/urdf/wheel_chair.urdf (robot description, URDF)
Before this commit: robot wheel_chair, 23 links, 22 joints
Joints:
- joint base_joint: origin xyz=0.0 0.0 0.15345 rpy=0 0 0 -> xyz=-0.40 0.0 0.15345 rpy=0 0 0

Commit message: Performansı en optimize hale getirilmiş durum, çekim bu parametreler ile yapıldı.

File: wheel_chair/urdf/wheel_chair.urdf (robot description, URDF)
Before this commit: robot wheel_chair, 23 links, 22 joints
Joints:
- joint base_joint: origin xyz=-0.40 0.0 0.15345 rpy=0 0 0 -> xyz=-0.35 0.0 0.15345 rpy=0 0 0

Commit message: gereksizler silindi

File: wheel_chair/urdf/wheel_chair.urdf (robot description, URDF)
Before this commit: robot wheel_chair, 23 links, 22 joints
Joints:
- joint base_joint: origin xyz=-0.35 0.0 0.15345 rpy=0 0 0 -> xyz=-0.40 0.0 0.15345 rpy=0 0 0

Commit message: kamera cikartildi, yeni harita eklendi, bazı ufak değişiklikler

File: wheel_chair/urdf/wheel_chair.urdf (robot description, URDF)
Before this commit: robot wheel_chair, 23 links, 22 joints
Links:
- removed link camera_accel_frame
- removed link camera_accel_optical_frame
- removed link camera_color_frame
- removed link camera_color_optical_frame
- removed link camera_depth_frame
- removed link camera_depth_optical_frame
- removed link camera_gyro_frame
- removed link camera_gyro_optical_frame
- removed link camera_imu_optical_frame
- removed link camera_infra1_frame
- removed link camera_infra1_optical_frame
- removed link camera_infra2_frame
- removed link camera_infra2_optical_frame
- removed link camera_link
Joints:
- removed joint camera_accel_joint
- removed joint camera_accel_optical_joint
- removed joint camera_color_joint
- removed joint camera_color_optical_joint
- removed joint camera_depth_joint
- removed joint camera_depth_optical_joint
- removed joint camera_gyro_joint
- removed joint camera_gyro_optical_joint
- removed joint camera_imu_optical_joint
- removed joint camera_infra1_joint
- removed joint camera_infra1_optical_joint
- removed joint camera_infra2_joint
- removed joint camera_infra2_optical_joint
- removed joint camera_joint
- joint base_joint: origin xyz=-0.40 0.0 0.15345 rpy=0 0 0 -> xyz=0.0 0.0 0.0 rpy=0 0 0

Commit message: trajectoryplannerros calisiyor, izin oncesi son commit

File: wheel_chair/urdf/wheel_chair.urdf (robot description, URDF)
Before this commit: robot wheel_chair, 9 links, 8 joints
Joints:
- joint base_joint: origin xyz=0.0 0.0 0.0 rpy=0 0 0 -> xyz=-0.40 0.0 0.15345 rpy=0 0 0
